File: examples/buck_imu/buck_imu.kicad_sch (KiCad schematic)
At the start: 16 parts, among them J1 USB_C, U1 ESP32-S3, U2 TPS62160, U3 ICM42688, U4 USBLC6, Y1 40MHz

Commit message: fix(validation): enforce fail-fast footprint resolution
- Remove silent footprint and pad recovery paths
- Reject unresolved footprints instead of guessing
- Add pad_count_mismatch validation
- Surface all footprint validation errors in a single report
- Ensure Layla never invents electrical connectivity
Parts:
- C1: symbol C -> C_C1
- C2: symbol C -> C_C2
- C3: symbol C -> C_C3
- C4: symbol C -> C_C4
- C5: symbol C -> C_C5
- J1: symbol USB -> USB_J1
- L1: symbol L -> L_L1
- R1: symbol R -> R_R1
- R2: symbol R -> R_R2
- TP1: symbol TestPoint -> TestPoint_TP1
- TP2: symbol TestPoint -> TestPoint_TP2
- U1: symbol MCU -> MCU_U1
- U2: symbol Regulator -> Regulator_U2
- U3: symbol IMU -> IMU_U3
- U4: symbol Diode -> Diode_U4
- Y1: symbol Crystal -> Crystal_Y1
Changed lines of the file:
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@@
   )
   (symbol
-    (lib_id "MCU")
+    (lib_id "MCU_U1")
     (at 30 30 0)
     (unit 1)
@@
   )
   (symbol
-    (lib_id "Regulator")
+    (lib_id "Regulator_U2")
     (at 65 30 0)
     (unit 1)
@@
   )
   (symbol
-    (lib_id "L")
+    (lib_id "L_L1")
     (at 100 30 0)
     (unit 1)
@@
   )
   (symbol
-    (lib_id "C")
+    (lib_id "C_C1")
     (at 135 30 0)
     (unit 1)
@@
   )
   (symbol
-    (lib_id "C")
+    (lib_id "C_C2")
     (at 170 30 0)
     (unit 1)
@@
   )
   (symbol
-    (lib_id "R")
+    (lib_id "R_R1")
     (at 205 30 0)
     (unit 1)
@@
   )
   (symbol
-    (lib_id "R")
+    (lib_id "R_R2")
     (at 30 65 0)
     (unit 1)
@@
   )
   (symbol
-    (lib_id "C")
+    (lib_id "C_C3")
     (at 65 65 0)
     (unit 1)
@@
   )
   (symbol
-    (lib_id "C")
+    (lib_id "C_C4")
     (at 100 65 0)
     (unit 1)
@@
   )
   (symbol
-    (lib_id "USB")
+    (lib_id "USB_J1")
     (at 135 65 0)
     (unit 1)
@@
   )
   (symbol
-    (lib_id "Diode")
+    (lib_id "Diode_U4")
     (at 170 65 0)
     (unit 1)
@@
   )
   (symbol
-    (lib_id "IMU")
+    (lib_id "IMU_U3")
     (at 205 65 0)
     (unit 1)
@@
   )
   (symbol
-    (lib_id "C")
+    (lib_id "C_C5")
     (at 30 100 0)
     (unit 1)
@@
   )
   (symbol
-    (lib_id "Crystal")
+    (lib_id "Crystal_Y1")
     (at 65 100 0)
     (unit 1)
@@
   )
   (symbol
-    (lib_id "TestPoint")
+    (lib_id "TestPoint_TP1")
     (at 100 100 0)
     (unit 1)
@@
   )
   (symbol
-    (lib_id "TestPoint")
+    (lib_id "TestPoint_TP2")
     (at 135 100 0)
     (unit 1)
