File: examples/mainboard/mainboard.kicad_sch (KiCad schematic)
At the start: 187 parts, among them J10 MOT0, J11 MOT1, J12 MOT2, J13 MOT3, J20 VMOT_IN, J21 12V_IN, J30 RJ45, J31 CAN, J32 RS485, J33 USB_C, J40 GPIO-A, J41 SWD, J42 ADC, Q1 CSD18540, Q10 CSD18540, Q11 CSD18540, Q12 CSD18540, Q13 CSD18540, Q14 CSD18540, Q15 CSD18540, Q16 CSD18540, Q17 CSD18540, Q18 CSD18540, Q19 CSD18540, Q2 CSD18540, Q20 CSD18540, Q21 CSD18540, Q22 CSD18540, Q23 CSD18540, Q24 CSD18540, Q3 CSD18540, Q4 CSD18540, Q5 CSD18540, Q6 CSD18540, Q7 CSD18540, Q8 CSD18540, Q9 CSD18540, U1 AM62 SoC, U10 TPS5450 5V, U11 TPS62 3V3, U12 TPS62 1V8, U13 TPS62 1V2, U14 TPS54 0V8, U15 LP5907 3V3A, U2 RP2040 coproc, U20 DRV8353 ch0, U21 DRV8353 ch1, U22 DRV8353 ch2, U23 DRV8353 ch3, U3 ICE40 FPGA, U4 W25Q flash, U40 ICM42688 imu, U41 BMI270 imu, U42 MMC5983 mag, U43 BMP390 baro, U44 SHT45 rh, U45 VL53 tof, U46 ADS131 adc, U47 MAX31855 tc, U5 LPDDR4, U50 nRF52840, U51 SX1262 LoRa, U6 LPDDR4, U60 DP83825 PHY, U61 TCAN332, U62 THVD1500 485, U63 TPD4S ESD, Y1 25MHz, Y2 32.768k, Y3 50MHz eth

Commit message: fix(validation): enforce fail-fast footprint resolution
- Remove silent footprint and pad recovery paths
- Reject unresolved footprints instead of guessing
- Add pad_count_mismatch validation
- Surface all footprint validation errors in a single report
- Ensure Layla never invents electrical connectivity
Parts:
- ANT0: symbol Antenna -> Antenna_ANT0
- ANT1: symbol Antenna -> Antenna_ANT1
- C101: symbol C -> C_C101
- C102: symbol C -> C_C102
- C103: symbol C -> C_C103
- C104: symbol C -> C_C104
- C105: symbol C -> C_C105
- C106: symbol C -> C_C106
- C107: symbol C -> C_C107
- C108: symbol C -> C_C108
- C109: symbol C -> C_C109
- C110: symbol C -> C_C110
- C111: symbol C -> C_C111
- C112: symbol C -> C_C112
- C113: symbol C -> C_C113
- C114: symbol C -> C_C114
- C115: symbol C -> C_C115
- C116: symbol C -> C_C116
- C117: symbol C -> C_C117
- C118: symbol C -> C_C118
- C119: symbol C -> C_C119
- C120: symbol C -> C_C120
- C121: symbol C -> C_C121
- C122: symbol C -> C_C122
- C123: symbol C -> C_C123
- C124: symbol C -> C_C124
- C125: symbol C -> C_C125
- C126: symbol C -> C_C126
- C127: symbol C -> C_C127
- C128: symbol C -> C_C128
- C129: symbol C -> C_C129
- C130: symbol C -> C_C130
- C131: symbol C -> C_C131
- C132: symbol C -> C_C132
- C133: symbol C -> C_C133
- C134: symbol C -> C_C134
- C135: symbol C -> C_C135
- C136: symbol C -> C_C136
- C137: symbol C -> C_C137
- C138: symbol C -> C_C138
- C139: symbol C -> C_C139
- C140: symbol C -> C_C140
- C141: symbol C -> C_C141
- C142: symbol C -> C_C142
- C143: symbol C -> C_C143
- C144: symbol C -> C_C144
- C200: symbol C -> C_C200
- C201: symbol C -> C_C201
- C202: symbol C -> C_C202
- C203: symbol C -> C_C203
- C204: symbol C -> C_C204
- C205: symbol C -> C_C205
- C206: symbol C -> C_C206
- C207: symbol C -> C_C207
- C208: symbol C -> C_C208
- C209: symbol C -> C_C209
- C220: symbol C -> C_C220
- C221: symbol C -> C_C221
- C222: symbol C -> C_C222
- C223: symbol C -> C_C223
- C224: symbol C -> C_C224
- C225: symbol C -> C_C225
- C226: symbol C -> C_C226
- C227: symbol C -> C_C227
- C240: symbol C -> C_C240
- C241: symbol C -> C_C241
- D1: symbol D -> D_D1
- D2: symbol D -> D_D2
- D3: symbol D -> D_D3
- D4: symbol D -> D_D4
- D5: symbol D -> D_D5
- D6: symbol D -> D_D6
- D7: symbol D -> D_D7
- D8: symbol D -> D_D8
- J10: symbol Conn -> Conn_J10
- J11: symbol Conn -> Conn_J11
- J12: symbol Conn -> Conn_J12
- J13: symbol Conn -> Conn_J13
- J20: symbol Conn -> Conn_J20
- J21: symbol Conn -> Conn_J21
- J30: symbol Conn -> Conn_J30
- J31: symbol Conn -> Conn_J31
- J32: symbol Conn -> Conn_J32
- J33: symbol USB -> USB_J33
- J40: symbol Conn -> Conn_J40
- J41: symbol Conn -> Conn_J41
- J42: symbol Conn -> Conn_J42
- L1: symbol L -> L_L1
- L2: symbol L -> L_L2
- L20: symbol L -> L_L20
- L21: symbol L -> L_L21
- L3: symbol L -> L_L3
- L4: symbol L -> L_L4
- L5: symbol L -> L_L5
- Q1: symbol Q -> Q_Q1
- Q10: symbol Q -> Q_Q10
- Q11: symbol Q -> Q_Q11
- Q12: symbol Q -> Q_Q12
- Q13: symbol Q -> Q_Q13
- Q14: symbol Q -> Q_Q14
- Q15: symbol Q -> Q_Q15
- Q16: symbol Q -> Q_Q16
- Q17: symbol Q -> Q_Q17
- Q18: symbol Q -> Q_Q18
- Q19: symbol Q -> Q_Q19
- Q2: symbol Q -> Q_Q2
- Q20: symbol Q -> Q_Q20
- Q21: symbol Q -> Q_Q21
- Q22: symbol Q -> Q_Q22
- Q23: symbol Q -> Q_Q23
- Q24: symbol Q -> Q_Q24
- Q3: symbol Q -> Q_Q3
- Q4: symbol Q -> Q_Q4
- Q5: symbol Q -> Q_Q5
- Q6: symbol Q -> Q_Q6
- Q7: symbol Q -> Q_Q7
- Q8: symbol Q -> Q_Q8
- Q9: symbol Q -> Q_Q9
- R1: symbol R -> R_R1
- R10: symbol R -> R_R10
- R11: symbol R -> R_R11
- R12: symbol R -> R_R12
- R13: symbol R -> R_R13
- R14: symbol R -> R_R14
- R15: symbol R -> R_R15
- R16: symbol R -> R_R16
- R17: symbol R -> R_R17
- R18: symbol R -> R_R18
- R19: symbol R -> R_R19
- R2: symbol R -> R_R2
- R20: symbol R -> R_R20
- R21: symbol R -> R_R21
- R22: symbol R -> R_R22
- R23: symbol R -> R_R23
- R24: symbol R -> R_R24
- R25: symbol R -> R_R25
- R26: symbol R -> R_R26
- R27: symbol R -> R_R27
- R28: symbol R -> R_R28
- R29: symbol R -> R_R29
- R3: symbol R -> R_R3
- R30: symbol R -> R_R30
- R31: symbol R -> R_R31
- R32: symbol R -> R_R32
- R4: symbol R -> R_R4
- R5: symbol R -> R_R5
- R6: symbol R -> R_R6
- R7: symbol R -> R_R7
- R8: symbol R -> R_R8
- R9: symbol R -> R_R9
- TP1: symbol TestPoint -> TestPoint_TP1
- TP2: symbol TestPoint -> TestPoint_TP2
- TP3: symbol TestPoint -> TestPoint_TP3
- TP4: symbol TestPoint -> TestPoint_TP4
- U1: symbol MCU -> MCU_U1
- U10: symbol Regulator -> Regulator_U10
- U11: symbol Regulator -> Regulator_U11
- U12: symbol Regulator -> Regulator_U12
- U13: symbol Regulator -> Regulator_U13
- U14: symbol Regulator -> Regulator_U14
- U15: symbol Regulator -> Regulator_U15
- U2: symbol MCU -> MCU_U2
- U20: symbol MotorDriver -> MotorDriver_U20
- U21: symbol MotorDriver -> MotorDriver_U21
- U22: symbol MotorDriver -> MotorDriver_U22
- U23: symbol MotorDriver -> MotorDriver_U23
- U3: symbol MCU -> MCU_U3
- U4: symbol Sensor -> Sensor_U4
- U40: symbol Sensor -> Sensor_U40
- U41: symbol Sensor -> Sensor_U41
- U42: symbol Sensor -> Sensor_U42
- U43: symbol Sensor -> Sensor_U43
- U44: symbol Sensor -> Sensor_U44
- U45: symbol Sensor -> Sensor_U45
- U46: symbol Sensor -> Sensor_U46
- U47: symbol Sensor -> Sensor_U47
- U5: symbol MCU -> MCU_U5
- U50: symbol RF -> RF_U50
- U51: symbol RF -> RF_U51
- U6: symbol MCU -> MCU_U6
- U60: symbol MCU -> MCU_U60
- U61: symbol Sensor -> Sensor_U61
- U62: symbol Sensor -> Sensor_U62
- U63: symbol Diode -> Diode_U63
- Y1: symbol Crystal -> Crystal_Y1
- Y2: symbol Crystal -> Crystal_Y2
- Y3: symbol Crystal -> Crystal_Y3
Connections:
- net 1V2: now also U3.8, U5.12, U5.14, U5.16, U6.12, U6.14, U6.16, U60.11; no longer U3.20, U5.22, U5.44, U5.46, U6.22, U6.44, U6.46, U60.47
- net 3V3: now also J30.5, U15.2, U2.12, U3.6, U60.8, U60.9; no longer U2.22, U3.18, U60.20, U60.45
- net 3V3A: now also U42.2, U43.2, U44.2, U45.2; no longer U42.3, U43.3, U44.3, U45.3
- net ADC0: now also U2.16; no longer U2.46
- net ADC1: now also U2.15; no longer U2.45
- net ADC2: now also J42.4, U2.14; no longer U2.44
- net ADC3: now also U2.13; no longer U2.43
- net CS_FPGA: now also U3.5; no longer U3.17
- net DCLK: now also U3.9, U5.18, U6.18; no longer U3.45, U5.48, U6.48
- net DCLKN: now also U5.17, U6.17; no longer U5.47, U6.47
- net DQ0: now also U3.13, U5.10, U6.10; no longer U3.49, U5.20, U6.20
- net DQ1: now also U3.12, U5.9, U6.9; no longer U3.48, U5.19, U6.19
- net DQ10: now also U5.24, U6.24; no longer U5.54, U6.54
- net DQ11: now also U5.23, U6.23; no longer U5.53, U6.53
- net DQ12: now also U5.22, U6.22; no longer U5.52, U6.52
- net DQ13: now also U5.21, U6.21; no longer U5.51, U6.51
- net DQ14: now also U5.20, U6.20; no longer U5.50, U6.50
- net DQ15: now also U5.19, U6.19; no longer U5.49, U6.49
- net DQ2: now also U3.11, U5.8, U6.8; no longer U3.47, U5.18, U6.18
- net DQ3: now also U3.10, U5.7, U6.7; no longer U3.46, U5.17, U6.17
- net DQ4: now also U5.6, U6.6; no longer U5.16, U6.16
- net DQ5: now also U5.5, U6.5; no longer U5.15, U6.15
- net DQ6: now also U5.4, U6.4; no longer U5.14, U6.14
- net DQ7: now also U5.3, U6.3; no longer U5.13, U6.13
- net DQ8: now also U5.2, U6.2; no longer U5.12, U6.12
- net DQ9: now also U5.1, U6.1; no longer U5.11, U6.11
- net ETH_RXN: now also J30.6, U60.15; no longer U60.51
- net ETH_RXP: now also J30.1, U60.16; no longer U60.52
- net ETH_TXN: now also J30.2, U60.1; no longer U60.13
- net ETH_TXP: now also J30.3, U60.2; no longer U60.14
- net FAB0: now also U2.3, U3.1; no longer U2.13, U3.13
- net FAB1: now also U2.2, U3.16; no longer U2.12, U3.52
- net FAB2: now also U2.1, U3.15; no longer U2.11, U3.51
- net FAB3: now also U2.24, U3.14; no longer U2.54, U3.50
- net GND: now also J21.2, J30.4, J31.4, J32.4, J40.4, U15.1, U2.11, U3.7, U42.1, U43.1, U44.1, U45.1, U5.11, U5.13, U5.15, U6.11, U6.13, U6.15, U60.10, U60.7; no longer U2.21, U3.19, U42.2, U43.2, U44.2, U45.2, U5.21, U5.43, U5.45, U6.21, U6.43, U6.45, U60.19, U60.46
- net GPIO0: now also J40.3
- net GPIO1: now also J40.2
- net GPIO2: now also J40.1
- net GPIO3: now also J40.6
- net GPIO4: now also J40.5
- net GPIO5: now also U2.23; no longer U2.53
- net GPIO6: now also U2.22; no longer U2.52
- net GPIO7: now also U2.21; no longer U2.51
- net MDC: now also U60.14; no longer U60.50
- net MDIO: now also U60.13; no longer U60.49
- net MISO: now also U2.8, U3.2; no longer U2.18, U3.14
- net MOSI: now also U2.9, U3.3; no longer U2.19, U3.15, U40.8, U41.8, U46.8, U47.8
- net PGND: now also J20.2
- net PWM0: now also U2.20; no longer U2.50
- net PWM1: now also U2.19; no longer U2.49
- net PWM2: now also U2.18; no longer U2.48
- net PWM3: now also U2.17; no longer U2.47
- net RGMII_RX0: now also U60.4; no longer U60.16
- net RGMII_RX1: now also U60.3; no longer U60.15
- net RGMII_TX0: now also U60.6; no longer U60.18
- net RGMII_TX1: now also U60.5; no longer U60.17
- net SCK: now also U2.10, U3.4; no longer U2.20, U3.16
- net SCL: now also U2.6, U42.3, U43.3, U44.3, U45.3; no longer U2.16, U42.6, U43.6, U44.6, U45.6
- net SDA: now also U2.7, U42.4, U43.4, U44.4, U45.4; no longer U2.17, U42.7, U43.7, U44.7, U45.7
- net SWCLK: now also J41.4
- net UART1_RX: now also U2.4; no longer U2.14
- net UART1_TX: now also U2.5; no longer U2.15
- net VIN12: now also J21.1
- net VMOT: now also J20.1
- net XTAL1: now also U60.12; no longer U60.48
