File: examples/motor_driver/motor_driver.kicad_sch (KiCad schematic)
At the start: 13 parts, among them J1 PWR, J2 MOTOR, J3 USB_C, Q1 NMOS, U1 STM32G0, U2 DRV8313, U3 TPS54331, U4 INA240

Commit message: fix(validation): enforce fail-fast footprint resolution
- Remove silent footprint and pad recovery paths
- Reject unresolved footprints instead of guessing
- Add pad_count_mismatch validation
- Surface all footprint validation errors in a single report
- Ensure Layla never invents electrical connectivity
Parts:
- C1: symbol C -> C_C1
- C2: symbol C -> C_C2
- C3: symbol C -> C_C3
- C4: symbol C -> C_C4
- J1: symbol Conn -> Conn_J1
- J2: symbol Conn -> Conn_J2
- J3: symbol USB -> USB_J3
- L1: symbol L -> L_L1
- Q1: symbol Mosfet -> Mosfet_Q1
- U1: symbol MCU -> MCU_U1
- U2: symbol MotorDriver -> MotorDriver_U2
- U3: symbol Regulator -> Regulator_U3
- U4: symbol ADC -> ADC_U4
Connections:
- net MOTOR_A: now also J2.2
- net MOTOR_B: now also J2.1
Changed lines of the file:
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@@
   )
   (symbol
-    (lib_id "MCU")
+    (lib_id "MCU_U1")
     (at 30 30 0)
     (unit 1)
@@
   )
   (symbol
-    (lib_id "MotorDriver")
+    (lib_id "MotorDriver_U2")
     (at 65 30 0)
     (unit 1)
@@
   )
   (symbol
-    (lib_id "Regulator")
+    (lib_id "Regulator_U3")
     (at 100 30 0)
     (unit 1)
@@
   )
   (symbol
-    (lib_id "L")
+    (lib_id "L_L1")
     (at 135 30 0)
     (unit 1)
@@
   )
   (symbol
-    (lib_id "C")
+    (lib_id "C_C1")
     (at 170 30 0)
     (unit 1)
@@
   )
   (symbol
-    (lib_id "C")
+    (lib_id "C_C2")
     (at 205 30 0)
     (unit 1)
@@
   )
   (symbol
-    (lib_id "Mosfet")
+    (lib_id "Mosfet_Q1")
     (at 30 65 0)
     (unit 1)
@@
   )
   (symbol
-    (lib_id "Conn")
+    (lib_id "Conn_J1")
     (at 65 65 0)
     (unit 1)
@@
   )
   (symbol
-    (lib_id "Conn")
+    (lib_id "Conn_J2")
     (at 100 65 0)
     (unit 1)
@@
   )
   (symbol
-    (lib_id "ADC")
+    (lib_id "ADC_U4")
     (at 135 65 0)
     (unit 1)
@@
   )
   (symbol
-    (lib_id "C")
+    (lib_id "C_C3")
     (at 170 65 0)
     (unit 1)
@@
   )
   (symbol
-    (lib_id "C")
+    (lib_id "C_C4")
     (at 205 65 0)
     (unit 1)
@@
   )
   (symbol
-    (lib_id "USB")
+    (lib_id "USB_J3")
     (at 30 100 0)
     (unit 1)
