File: examples/rf_sensor/rf_sensor.kicad_sch (KiCad schematic)
At the start: 13 parts, among them J1 BATT, U1 nRF52840, U2 MP2359, U3 BME280, Y1 32MHz

Commit message: fix(validation): enforce fail-fast footprint resolution
- Remove silent footprint and pad recovery paths
- Reject unresolved footprints instead of guessing
- Add pad_count_mismatch validation
- Surface all footprint validation errors in a single report
- Ensure Layla never invents electrical connectivity
Parts:
- ANT1: symbol Antenna -> Antenna_ANT1
- C1: symbol C -> C_C1
- C2: symbol C -> C_C2
- C3: symbol C -> C_C3
- C4: symbol C -> C_C4
- J1: symbol Conn -> Conn_J1
- L1: symbol L -> L_L1
- R1: symbol R -> R_R1
- R2: symbol R -> R_R2
- U1: symbol MCU -> MCU_U1
- U2: symbol Regulator -> Regulator_U2
- U3: symbol Sensor -> Sensor_U3
- Y1: symbol Crystal -> Crystal_Y1
Changed lines of the file:
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@@
   )
   (symbol
-    (lib_id "MCU")
+    (lib_id "MCU_U1")
     (at 30 30 0)
     (unit 1)
@@
   )
   (symbol
-    (lib_id "Antenna")
+    (lib_id "Antenna_ANT1")
     (at 65 30 0)
     (unit 1)
@@
   )
   (symbol
-    (lib_id "Regulator")
+    (lib_id "Regulator_U2")
     (at 100 30 0)
     (unit 1)
@@
   )
   (symbol
-    (lib_id "L")
+    (lib_id "L_L1")
     (at 135 30 0)
     (unit 1)
@@
   )
   (symbol
-    (lib_id "C")
+    (lib_id "C_C1")
     (at 170 30 0)
     (unit 1)
@@
   )
   (symbol
-    (lib_id "C")
+    (lib_id "C_C2")
     (at 205 30 0)
     (unit 1)
@@
   )
   (symbol
-    (lib_id "Sensor")
+    (lib_id "Sensor_U3")
     (at 30 65 0)
     (unit 1)
@@
   )
   (symbol
-    (lib_id "C")
+    (lib_id "C_C3")
     (at 65 65 0)
     (unit 1)
@@
   )
   (symbol
-    (lib_id "C")
+    (lib_id "C_C4")
     (at 100 65 0)
     (unit 1)
@@
   )
   (symbol
-    (lib_id "Crystal")
+    (lib_id "Crystal_Y1")
     (at 135 65 0)
     (unit 1)
@@
   )
   (symbol
-    (lib_id "Conn")
+    (lib_id "Conn_J1")
     (at 170 65 0)
     (unit 1)
@@
   )
   (symbol
-    (lib_id "R")
+    (lib_id "R_R1")
     (at 205 65 0)
     (unit 1)
@@
   )
   (symbol
-    (lib_id "R")
+    (lib_id "R_R2")
     (at 30 100 0)
     (unit 1)
