File: examples/robot_soc/robot_soc.kicad_sch (KiCad schematic)
At the start: 72 parts, among them J1 USB_C, J2 MOTOR, J3 SWD, J4 GPIO, J5 VMOT_IN, J6 CAN, J7 UART, Q1 CSD18540, Q2 CSD18540, Q3 CSD18540, Q4 CSD18540, Q5 CSD18540, Q6 CSD18540, U1 STM32H743 MCU, U10 MMC5983 mag, U11 BMP390 baro, U12 ADS131 ADC, U13 TCAN332, U2 TPS54560 5V, U3 TPS62912 3V3, U4 TLV62568 1V8, U5 LP5907 3V3A, U6 TPD4S ESD, U7 DRV8353 gate, U8 nRF52840, U9 ICM42688 IMU, Y1 25MHz, Y2 32.768kHz

Commit message: fix(validation): enforce fail-fast footprint resolution
- Remove silent footprint and pad recovery paths
- Reject unresolved footprints instead of guessing
- Add pad_count_mismatch validation
- Surface all footprint validation errors in a single report
- Ensure Layla never invents electrical connectivity
Parts:
- ANT1: symbol Antenna -> Antenna_ANT1
- C1: symbol C -> C_C1
- C101: symbol C -> C_C101
- C102: symbol C -> C_C102
- C103: symbol C -> C_C103
- C104: symbol C -> C_C104
- C105: symbol C -> C_C105
- C106: symbol C -> C_C106
- C107: symbol C -> C_C107
- C108: symbol C -> C_C108
- C109: symbol C -> C_C109
- C110: symbol C -> C_C110
- C111: symbol C -> C_C111
- C112: symbol C -> C_C112
- C113: symbol C -> C_C113
- C114: symbol C -> C_C114
- C115: symbol C -> C_C115
- C116: symbol C -> C_C116
- C2: symbol C -> C_C2
- C20: symbol C -> C_C20
- C21: symbol C -> C_C21
- C3: symbol C -> C_C3
- C30: symbol C -> C_C30
- C4: symbol C -> C_C4
- C5: symbol C -> C_C5
- D1: symbol D -> D_D1
- D2: symbol D -> D_D2
- J1: symbol USB -> USB_J1
- J2: symbol Conn -> Conn_J2
- J3: symbol Conn -> Conn_J3
- J4: symbol Conn -> Conn_J4
- J5: symbol Conn -> Conn_J5
- J6: symbol Conn -> Conn_J6
- J7: symbol Conn -> Conn_J7
- L1: symbol L -> L_L1
- L2: symbol L -> L_L2
- L3: symbol L -> L_L3
- L4: symbol L -> L_L4
- Q1: symbol Q -> Q_Q1
- Q2: symbol Q -> Q_Q2
- Q3: symbol Q -> Q_Q3
- Q4: symbol Q -> Q_Q4
- Q5: symbol Q -> Q_Q5
- Q6: symbol Q -> Q_Q6
- R1: symbol R -> R_R1
- R10: symbol R -> R_R10
- R11: symbol R -> R_R11
- R12: symbol R -> R_R12
- R13: symbol R -> R_R13
- R2: symbol R -> R_R2
- R3: symbol R -> R_R3
- R4: symbol R -> R_R4
- R5: symbol R -> R_R5
- R6: symbol R -> R_R6
- R7: symbol R -> R_R7
- TP1: symbol TestPoint -> TestPoint_TP1
- TP2: symbol TestPoint -> TestPoint_TP2
- U1: symbol MCU -> MCU_U1
- U10: symbol Sensor -> Sensor_U10
- U11: symbol Sensor -> Sensor_U11
- U12: symbol ADC -> ADC_U12
- U13: symbol Sensor -> Sensor_U13
- U2: symbol Regulator -> Regulator_U2
- U3: symbol Regulator -> Regulator_U3
- U4: symbol Regulator -> Regulator_U4
- U5: symbol Regulator -> Regulator_U5
- U6: symbol Diode -> Diode_U6
- U7: symbol MotorDriver -> MotorDriver_U7
- U8: symbol RF -> RF_U8
- U9: symbol IMU -> IMU_U9
- Y1: symbol Crystal -> Crystal_Y1
- Y2: symbol Crystal -> Crystal_Y2
Connections:
- net 3V3: now also J7.4, U5.2
- net 5V: now also U13.2, U13.6; no longer U13.1, U13.3
- net CANH: now also U13.7; no longer U13.4
- net CANL: now also U13.8
- net CANRX: now also U13.1
- net CANTX: now also U13.4
- net GND: now also J4.4, J6.4, U13.3, U13.5, U5.1; no longer U13.2
- net GPIO0: now also J4.3
- net GPIO1: now also J4.2
- net GPIO2: now also J4.1
- net GPIO3: now also J4.6
- net GPIO4: now also J4.5
- net PGND: now also J5.2
- net SWCLK: now also J3.4
- net VMOT: now also J5.1
